File: pcb/interfaces.kicad_sch (KiCad schematic)
At the start: 5 parts

Commit message: Added labels for sensors
Fixed part numbers for connectors
Remove unnecessary property values
Parts:
- J2: Digikey 455-BM04B-SRSS-TBTR-ND -> 455-SM04B-SRSS-TBTR-ND; Mouser 306-BM04BSRSSTBTLFSN -> 306-SM04BSRSSTBTLFSN
Changed lines of the file:
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@@
-			)
-		)
-		(property "ALT_LCSC" ""
-			(at 60.96 57.15 90)
-			(effects
-				(font
-					(size 1.27 1.27)
-				)
-				(hide yes)
-			)
-		)
-		(property "ALT_LCSC_2" ""
-			(at 60.96 57.15 90)
-			(effects
-				(font
-					(size 1.27 1.27)
-				)
-				(hide yes)
-			)
-		)
-		(property "ALT_MN" ""
-			(at 60.96 57.15 90)
-			(effects
-				(font
-					(size 1.27 1.27)
-				)
-				(hide yes)
-			)
-		)
-		(property "ALT_MPN" ""
-			(at 60.96 57.15 90)
-			(effects
-				(font
-					(size 1.27 1.27)
-				)
-				(hide yes)
 			)
 		)
@@
 			)
 		)
-		(property "ALT_LCSC" ""
-			(at 41.91 55.88 0)
-			(effects
-				(font
-					(size 1.27 1.27)
-				)
-				(hide yes)
-			)
-		)
-		(property "ALT_LCSC_2" ""
-			(at 41.91 55.88 0)
-			(effects
-				(font
-					(size 1.27 1.27)
-				)
-				(hide yes)
-			)
-		)
-		(property "ALT_MN" ""
-			(at 41.91 55.88 0)
-			(effects
-				(font
-					(size 1.27 1.27)
-				)
-				(hide yes)
-			)
-		)
-		(property "ALT_MPN" ""
-			(at 41.91 55.88 0)
-			(effects
-				(font
-					(size 1.27 1.27)
-				)
-				(hide yes)
-			)
-		)
 		(pin "1"
 		)
@@
 			)
 		)
-		(property "Mouser" "306-BM04BSRSSTBTLFSN"
+		(property "Mouser" "306-SM04BSRSSTBTLFSN"
 			(at 46.99 52.578 0)
 			(effects
@@
 			)
 		)
-		(property "Digikey" "455-BM04B-SRSS-TBTR-ND"
+		(property "Digikey" "455-SM04B-SRSS-TBTR-ND"
 			(at 47.498 54.61 0)
 			(effects
@@
 		(property "LCSC" "C2763614"
 			(at 46.736 56.642 0)
-			(effects
-				(font
-					(size 1.27 1.27)
-				)
-				(hide yes)
-			)
-		)
-		(property "ALT_LCSC" ""
-			(at 41.91 30.48 0)
-			(effects
-				(font
-					(size 1.27 1.27)
-				)
-				(hide yes)
-			)
-		)
-		(property "ALT_LCSC_2" ""
-			(at 41.91 30.48 0)
-			(effects
-				(font
-					(size 1.27 1.27)
-				)
-				(hide yes)
-			)
-		)
-		(property "ALT_MN" ""
-			(at 41.91 30.48 0)
-			(effects
-				(font
-					(size 1.27 1.27)
-				)
-				(hide yes)
-			)
-		)
-		(property "ALT_MPN" ""
-			(at 41.91 30.48 0)
 			(effects
 				(font
@@
 			)
 		)
-		(property "ALT_LCSC" ""
-			(at 121.92 43.18 0)
-			(effects
-				(font
-					(size 1.27 1.27)
-				)
-				(hide yes)
-			)
-		)
-		(property "ALT_LCSC_2" ""
-			(at 121.92 43.18 0)
-			(effects
-				(font
-					(size 1.27 1.27)
-				)
-				(hide yes)
-			)
-		)
-		(property "ALT_MN" ""
-			(at 121.92 43.18 0)
-			(effects
-				(font
-					(size 1.27 1.27)
-				)
-				(hide yes)
-			)
-		)
-		(property "ALT_MPN" ""
-			(at 121.92 43.18 0)
-			(effects
-				(font
-					(size 1.27 1.27)
-				)
-				(hide yes)
-			)
-		)
 		(pin "1"
 		)
@@
 			(effects
 				(font
-					(size 1.27 1.27)
-				)
-				(hide yes)
-			)
-		)
-		(property "ALT_LCSC" ""
-			(at 58.42 57.15 90)
-			(effects
-				(font
-					(size 1.27 1.27)
-				)
-				(hide yes)
-			)
-		)
-		(property "ALT_LCSC_2" ""
-			(at 58.42 57.15 90)
-			(effects
-				(font
-					(size 1.27 1.27)
-				)
-				(hide yes)
-			)
-		)
-		(property "ALT_MN" ""
-			(at 58.42 57.15 90)
-			(effects
-				(font
-					(size 1.27 1.27)
-				)
-				(hide yes)
-			)
-		)
-		(property "ALT_MPN" ""
-			(at 58.42 57.15 90)
-			(effects
-				(font

Commit message: Updated UPDI Connector
Integrated serial and UPDI
Changed to vertical connectors
Updated renders
Rounded cutouts
Adjusted silkscreen
Parts:
- removed J4: ~, CRGM Connector:JST_SH_BM03B-SRSS-TB_1x03-1MP_P1.00mm_Vertical, symbol CRGM Connector:JST-SH-3
- J2, J3: footprint CRGM Connector:JST_SH_SM04B-SRSS-TB_1x04-1MP_P1.00mm_Horizontal -> CRGM Connector:JST_SH_BM04B-SRSS-TB_1x04-1MP_P1.00mm_Vertical; Digikey 455-SM04B-SRSS-TBTR-ND -> 455-BM04B-SRSS-TBTR-ND; LCSC C2763614 -> C2919601; MPN SM04B-SRSS-TBT(LF)(SN) -> BM04B-SRSS-TBT(LF)(SN); Mouser 306-SM04BSRSSTBTLFSN -> 306-BM04BSRSSTBTLFSN
Connections:
- net GND: now also J2.0 (MP), J2.5 (MP), J3.0 (MP), J3.5 (MP)
Other:
- note removed: "Serial"
